Commit message: mira_robot finish

File: src/urdf_exam/urdf/mira_simple.urdf (robot description, URDF)
Before this commit: robot mira, 3 links, 2 joints
Links:
- added link camera_link; visual box size=0.0005 0.0005 0.0005
- added link head_link; visual mesh filename=package://urdf_exam/meshes/mira_head_v5.dae
- added link left_eye_link; visual mesh filename=package://urdf_exam/meshes/mira_eye_v4.dae
- added link right_eye_link; visual mesh filename=package://urdf_exam/meshes/mira_eye_v4.dae
- added link yaw_M3_link; visual cylinder length=0.005 radius=0.01
- link base_link: geometry visual mesh filename=package://urdf_exam/meshes/mira_body_v3.dae
Joints:
- added joint base_head_joint: type fixed, parent yaw_M3_link, child head_link, origin xyz=0 0 0 rpy=0 0 0
- added joint head_camera_joint: type fixed, parent head_link, child camera_link, origin xyz=0 0.057 0.0255 rpy=0 0 0
- added joint head_lefteye_joint: type fixed, parent head_link, child left_eye_link, origin xyz=0.0095 0.057 0.0085 rpy=-1.5708 0 0
- added joint head_righteye_joint: type fixed, parent head_link, child right_eye_link, origin xyz=-0.0095 0.057 0.0085 rpy=-1.5708 0 0
- added joint yaw_joint: type continuous, parent pitch_M2_link, child yaw_M3_link, origin xyz=0.01 0 0 rpy=0 1.5708 0, axis 0 0 1, limit effort=0.1 velocity=0.01
- joint roll_joint: origin xyz=0.0023 0 -0.005 rpy=0 0 0 -> xyz=0.0023 0 -0.0005 rpy=0 0 0
