Commit message: hector

File: src/mobile_robot/mobile_robot_description/urdf/mobile_robot.urdf (robot description, URDF)
Before this commit: robot mobile_robot, 5 links, 4 joints
Links:
- added link ar_camera_link
- added link ar_camera_link_tmp
Joints:
- added joint ar_camera_fixed_joint: type fixed, parent ar_camera_link_tmp, child ar_camera_link, origin xyz=0 0 0 rpy=0 0 -1.57
- added joint ar_camera_fixed_joint_tmp: type fixed, parent camera_link, child ar_camera_link_tmp, origin xyz=0 0 0 rpy=0 1.57 0
